Commit message: updates lab6

File: lab-6-dual-arm/models/ur5e.urdf (robot description, URDF)
Before this commit: robot ur5e, 9 links, 8 joints
Links:
- link base_link: mass 2.4429 -> 4.0; geometry 
- link ee_link: mass 0.0972 -> 0.1; geometry 
- link forearm_link: mass 3.0216 -> 2.275; geometry 
- link shoulder_link: mass 2.0736 -> 3.7; geometry 
- link upper_arm_link: mass 3.7887 -> 8.393; geometry 
- link wrist_1_link: mass 0.8128 -> 1.219; geometry 
- link wrist_2_link: mass 0.6150 -> 1.219; geometry 
- link wrist_3_link: mass 0.5593 -> 0.1889; geometry 
Joints:
- joint ee_fixed_joint: origin xyz=0 0 0.135 rpy=0 0 0 -> xyz=0 0.1 0 rpy=-1.5707963267948966 0 0
- joint elbow_joint: axis 0 0 1 -> 0 1 0; limit lower=-6.28318530718 upper=6.28318530718 effort=150.0 velocity=3.14 -> lower=-3.14159265359 upper=3.14159265359 effort=150.0 velocity=3.14; origin xyz=-0.425 0 0 rpy=0 0 0 -> xyz=0 -0.131 0.425 rpy=0 0 0
- joint shoulder_lift_joint: axis 0 0 1 -> 0 1 0; origin xyz=0 0 0 rpy=1.5707963267948966 0 0 -> xyz=0 0.138 0 rpy=0 1.5707963267948966 0
- joint shoulder_pan_joint: origin xyz=0 0 0.1625 rpy=0 0 0 -> xyz=0 0 0.163 rpy=0 0 0
- joint world_joint: origin xyz=0 0 0 rpy=0 0 0 -> xyz=0 0 0 rpy=0 0 3.14159265358979
- joint wrist_1_joint: axis 0 0 1 -> 0 1 0; origin xyz=-0.3922 0 0.1333 rpy=0 0 0 -> xyz=0 0 0.392 rpy=0 1.5707963267948966 0
- joint wrist_2_joint: origin xyz=0 0 0.0997 rpy=1.5707963267948966 0 0 -> xyz=0 0.127 0 rpy=0 0 0
- joint wrist_3_joint: axis 0 0 1 -> 0 1 0; origin xyz=0 0 0.0996 rpy=-1.5707963267948966 0 0 -> xyz=0 0 0.1 rpy=0 0 0
